Commit message: removed 'prefix'

File: urdf/mh24_macro.xacro (robot description, xacro)
@@ -4,5 +4,5 @@
 		<xacro:property name="pi" value="3.14159265358979323846264338327950288419716" />
 		<!-- link list -->
-		<link name="${prefix}base_link">
+		<link name="base_link">
 			<visual>
 				<geometry>
@@ -22,6 +22,6 @@
 			</collision>
 		</link>
-		<link name="${prefix}vendor_base_link" />
-		<link name="${prefix}link_s">
+		<link name="vendor_base_link" />
+		<link name="link_s">
 			<visual>
 				<geometry>
@@ -39,5 +39,5 @@
 			</collision>
 		</link>
-		<link name="${prefix}link_l">
+		<link name="link_l">
 			<visual>
 				<geometry>
@@ -53,5 +53,5 @@
 			</collision>
 		</link>
-		<link name="${prefix}link_u">
+		<link name="link_u">
 			<visual>
 				<geometry>
@@ -67,5 +67,5 @@
 			</collision>
 		</link>
-		<link name="${prefix}link_r">
+		<link name="link_r">
 			<visual>
 				<geometry>
@@ -81,5 +81,5 @@
 			</collision>
 		</link>
-		<link name="${prefix}link_b">
+		<link name="link_b">
 			<visual>
 				<geometry>
@@ -95,5 +95,5 @@
 			</collision>
 		</link>
-		<link name="${prefix}link_t">
+		<link name="link_t">
 			<visual>
 				<geometry>
@@ -109,29 +109,29 @@
 			</collision>
 		</link>
-		<link name="${prefix}vendor_ee" />
+		<link name="vendor_ee" />
 		<!-- end of link list -->
 		<!-- joint list -->
-		<joint name="${prefix}vendor_base_joint" type="fixed">
-			<parent link="${prefix}base_link" />
-			<child link="${prefix}vendor_base_link" />
+		<joint name="vendor_base_joint" type="fixed">
+			<parent link="base_link" />
+			<child link="vendor_base_link" />
 			<origin xyz="0 0 0.505" />
 		</joint>
-		<joint name="${prefix}joint_s" type="revolute">
-			<parent link="${prefix}base_link"/>
-			<child link="${prefix}link_s"/>
+		<joint name="joint_s" type="revolute">
+			<parent link="base_link"/>
+			<child link="link_s"/>
 			<origin xyz="0 0 0" />
 			<axis xyz="0 0 1" />
 			<limit lower="${-180 / 180.0 * pi}" upper="${180 / 180.0 * pi}" effort="100" velocity="3.44" />
 		</joint>
-		<joint name="${prefix}joint_l" type="revolute">
-			<parent link="${prefix}link_s"/>
-			<child link="${prefix}link_l"/>
+		<joint name="joint_l" type="revolute">
+			<parent link="link_s"/>
+			<child link="link_l"/>
 			<origin xyz="0.150 0 0.505" />
 			<axis xyz="0 1 0" />
 			<limit lower="${-105 / 180.0 * pi}" upper="${155 / 180.0 * pi}" effort="100" velocity="3.32" />
 		</joint>
-		<joint name="${prefix}joint_u" type="revolute">
-			<parent link="${prefix}link_l"/>
-			<child link="${prefix}link_u"/>
+		<joint name="joint_u" type="revolute">
+			<parent link="link_l"/>
+			<child link="link_u"/>
 			<origin xyz="0 0 0.760" />
 			<axis xyz="0 -1 0" />
@@ -139,28 +139,28 @@
 			<limit lower="${-86 / 180.0 * pi}" upper="${163 / 180.0 * pi}" effort="100" velocity="3.67" />
 		</joint>
-		<joint name="${prefix}joint_r" type="revolute">
-			<parent link="${prefix}link_u"/>
-			<child link="${prefix}link_r"/>
+		<joint name="joint_r" type="revolute">
+			<parent link="link_u"/>
+			<child link="link_r"/>
 			<origin xyz="0 0 0.200" />
 			<axis xyz="-1 0 0" />
 			<limit lower="${-200 / 180.0 * pi}" upper="${200 / 180.0 * pi}" effort="100" velocity="7.16" />
 		</joint>
-		<joint name="${prefix}joint_b" type="revolute">
-			<parent link="${prefix}link_r"/>
-			<child link="${prefix}link_b"/>
+		<joint name="joint_b" type="revolute">
+			<parent link="link_r"/>
+			<child link="link_b"/>
 			<origin xyz="0.795 0 0" />
 			<axis xyz="0 -1 0" />
 			<limit lower="${-150 / 180.0 * pi}" upper="${150 / 180.0 * pi}" effort="100" velocity="7.16" />
 		</joint>
-		<joint name="${prefix}joint_t" type="revolute">
-			<parent link="${prefix}link_b"/>
-			<child link="${prefix}link_t"/>
+		<joint name="joint_t" type="revolute">
+			<parent link="link_b"/>
+			<child link="link_t"/>
 			<origin xyz="0.100 0 0" />
 			<axis xyz="-1 0 0" />
 			<limit lower="${-455 / 180.0 * pi}" upper="${455 / 180.0 * pi}" effort="100" velocity="10.82" />
 		</joint>
-		<joint name="${prefix}vendor_ee_joint" type="fixed">
-			<parent link="${prefix}link_t" />
-			<child link="${prefix}vendor_ee" />
+		<joint name="vendor_ee_joint" type="fixed">
+			<parent link="link_t" />
+			<child link="vendor_ee" />
 			<origin rpy="0 ${-0.5 * pi} ${pi}" />
 		</joint>

Commit message: added number to joint

File: urdf/mh24_macro.xacro (robot description, xacro)
@@ -117,5 +117,5 @@
 			<origin xyz="0 0 0.505" />
 		</joint>
-		<joint name="joint_s" type="revolute">
+		<joint name="joint_1_s" type="revolute">
 			<parent link="base_link"/>
 			<child link="link_s"/>
@@ -124,5 +124,5 @@
 			<limit lower="${-180 / 180.0 * pi}" upper="${180 / 180.0 * pi}" effort="100" velocity="3.44" />
 		</joint>
-		<joint name="joint_l" type="revolute">
+		<joint name="joint_2_l" type="revolute">
 			<parent link="link_s"/>
 			<child link="link_l"/>
@@ -131,5 +131,5 @@
 			<limit lower="${-105 / 180.0 * pi}" upper="${155 / 180.0 * pi}" effort="100" velocity="3.32" />
 		</joint>
-		<joint name="joint_u" type="revolute">
+		<joint name="joint_3_u" type="revolute">
 			<parent link="link_l"/>
 			<child link="link_u"/>
@@ -139,5 +139,5 @@
 			<limit lower="${-86 / 180.0 * pi}" upper="${163 / 180.0 * pi}" effort="100" velocity="3.67" />
 		</joint>
-		<joint name="joint_r" type="revolute">
+		<joint name="joint_4_r" type="revolute">
 			<parent link="link_u"/>
 			<child link="link_r"/>
@@ -146,5 +146,5 @@
 			<limit lower="${-200 / 180.0 * pi}" upper="${200 / 180.0 * pi}" effort="100" velocity="7.16" />
 		</joint>
-		<joint name="joint_b" type="revolute">
+		<joint name="joint_5_b" type="revolute">
 			<parent link="link_r"/>
 			<child link="link_b"/>
@@ -153,5 +153,5 @@
 			<limit lower="${-150 / 180.0 * pi}" upper="${150 / 180.0 * pi}" effort="100" velocity="7.16" />
 		</joint>
-		<joint name="joint_t" type="revolute">
+		<joint name="joint_6_t" type="revolute">
 			<parent link="link_b"/>
 			<child link="link_t"/>

Commit message: deleted vendor_ee joint

File: urdf/mh24_macro.xacro (robot description, xacro)
@@ -109,5 +109,4 @@
 			</collision>
 		</link>
-		<link name="vendor_ee" />
 		<!-- end of link list -->
 		<!-- joint list -->
@@ -160,9 +159,4 @@
 			<limit lower="${-455 / 180.0 * pi}" upper="${455 / 180.0 * pi}" effort="100" velocity="10.82" />
 		</joint>
-		<joint name="vendor_ee_joint" type="fixed">
-			<parent link="link_t" />
-			<child link="vendor_ee" />
-			<origin rpy="0 ${-0.5 * pi} ${pi}" />
-		</joint>
 		<!-- end of joint list -->
 	</xacro:macro>

Commit message: deleted vendor_base_link

File: urdf/mh24_macro.xacro (robot description, xacro)
@@ -22,5 +22,4 @@
 			</collision>
 		</link>
-		<link name="vendor_base_link" />
 		<link name="link_s">
 			<visual>
@@ -111,9 +110,4 @@
 		<!-- end of link list -->
 		<!-- joint list -->
-		<joint name="vendor_base_joint" type="fixed">
-			<parent link="base_link" />
-			<child link="vendor_base_link" />
-			<origin xyz="0 0 0.505" />
-		</joint>
 		<joint name="joint_1_s" type="revolute">
 			<parent link="base_link"/>

Commit message: Changed robot color to blue

File: urdf/mh24_macro.xacro (robot description, xacro)
@@ -27,6 +27,6 @@
 					<mesh filename="package://yaskawa_mh24_support/meshes/mh24/visual/s_axis.stl"/>
 				</geometry>
-				<material name="silver">
-					<color rgba="0.8 0.8 0.8 1"/>
+				<material name="blue">
+					<color rgba="0 0 1 1"/>
 				</material>
 			</visual>
@@ -57,5 +57,5 @@
 					<mesh filename="package://yaskawa_mh24_support/meshes/mh24/visual/u_axis.stl"/>
 				</geometry>
-				<material name="silver"/>
+				<material name="blue"/>
 			</visual>
 			<collision>
@@ -85,5 +85,5 @@
 					<mesh filename="package://yaskawa_mh24_support/meshes/mh24/visual/b_axis.stl"/>
 				</geometry>
-				<material name="silver"/>
+				<material name="blue"/>
 			</visual>
 			<collision>
